File: corne-hotswap/corne-hotswap.kicad_pcb (KiCad board)
At the start: 2 copper layers, 133.2 x 90.7 mm, 56 parts, among them J1 Battery Connector, J2 nice!view, J3 OLED display, SW1 SW_Push, SW10 SW_Push, SW11 SW_Push, SW12 SW_Push, SW13 SW_Push, SW14 SW_Push, SW15 SW_Push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

Commit message: pcb edit
Parts:
- removed REF**: 1.5u, Project:1.5u
- added RSW1: SW_Push, Project:SW_PUSH_1P1T_6x3.5mm_H4.3_APEM_MJTP1243, F.Cu at (190.9, 0.20)
- JP10, JP7, JP8, JP9: moved to B.Cu
- PSW1: footprint Button_Switch_SMD:SW_SPDT_PCM12 -> Project:SW_SPDT_PCM12
- moved J2 183.6 mm to (164.6, 81.3)
- moved J3 181.5 mm to (164.6, 87.8)
- moved JP12 178.2 mm to (163.1, 77.3), turned to 90 degrees
- moved JP7 177.5 mm to (160.1, 77.3), turned to 90 degrees
- moved JP13 173.6 mm to (166.1, 77.3), turned to 90 degrees
- moved JP8 172.9 mm to (163.1, 77.3), turned to 90 degrees
- moved JP14 169.0 mm to (169.1, 77.3), turned to 90 degrees
- moved JP9 168.3 mm to (166.1, 77.3), turned to 90 degrees
- moved JP11 165.5 mm to (160.1, 77.3), turned to 90 degrees
- moved JP10 163.7 mm to (169.1, 77.3), turned to 90 degrees
- moved PSW1 134.0 mm to (164.6, 43.2), turned to 180 degrees
- moved U1 0.45 mm to (164.6, 60.0)
Connections:
- net raw renamed RAW
- U1 pad 12: unconnected-(U1-B5-Pad12) -> CS
- U1 pad 15: reset -> RST
- U1 pad 24: CS -> (no net)
Other:
- board size 133.2 x 90.7 mm -> 133.8 x 91.9 mm

Commit message: update
Parts:
- removed J3: OLED display, Project:OLED_Display
- removed JP10, JP11, JP12, JP13, JP14, JP7, JP8, JP9: SolderJumper_2_Open, Jumper:SolderJumper-2_P1.3mm_Open_RoundedPad1.0x1.5mm
- D1, D10, D11, D12, D13, D14, D15, D16, D17, D18, D19, D2, D20, D21, D3, D4, D5, D6, D7, D8, D9: footprint Project:Diode-Reversible -> Project:D_SOD-123F-Reversible
- moved D2 180.2 mm to (57.3, 77.3), turned to 180 degrees
- moved D3 180.2 mm to (57.3, 79.7), turned to 180 degrees
- moved D4 161.4 mm to (76.3, 58.4), turned to 180 degrees
- moved D5 160.8 mm to (76.3, 77.3), turned to 180 degrees
- moved D6 160.8 mm to (76.3, 79.7), turned to 180 degrees
- moved D9 154.9 mm to (95.3, 91.6), turned to 180 degrees
- moved D8 153.0 mm to (95.3, 72.6), turned to 180 degrees
- moved D7 144.8 mm to (95.3, 53.6), turned to 180 degrees
- moved D10 134.8 mm to (114.3, 51.2), turned to 180 degrees
- moved D12 134.3 mm to (114.3, 89.2), turned to 180 degrees
- moved D11 133.6 mm to (114.3, 70.2), turned to 180 degrees
- moved D13 125.0 mm to (123.8, 94.5), turned to 180 degrees
- moved D17 113.6 mm to (149.1, 98.9), turned to -90 degrees
- moved D21 100.5 mm to (158.6, 92.3), turned to -90 degrees
- moved D15 31.2 mm to (235.3, 82.4), turned to 180 degrees
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Connections:
- J2 pad 1: jump0 -> SDA
- J2 pad 2: jump1 -> SCL
- J2 pad 4: jump2 -> GND
- J2 pad 5: jump3 -> CS
- U1 pad 24: (no net) -> unconnected-(U1-B6-Pad24)

Commit message: edit
Parts:
- D1, D10, D11, D12, D13, D14, D15, D16, D17, D18, D19, D2, D20, D21, D3, D4, D5, D6, D7, D8, D9: footprint Project:D_SOD-123F-Reversible -> Project:D_SOD-123F-Reversible-Hotswap; moved to B.Cu
- moved D19 260.0 mm to (53.0, -117.2)
- moved D20 243.7 mm to (53.0, -97.0)
- moved D14 234.4 mm to (73.0, -97.0)
- moved D15 227.4 mm to (73.0, -77.0)
- moved D13 217.7 mm to (73.0, -117.2)
- moved D16 211.5 mm to (73.0, -56.9)
- moved D21 199.5 mm to (53.0, -77.0), turned to 180 degrees
- moved D18 184.8 mm to (73.0, -16.6)
- moved D2 183.2 mm to (113.2, -97.0)
- moved D7 170.8 mm to (93.2, -117.2)
- moved D8 169.7 mm to (93.2, -97.0)
- moved D9 168.6 mm to (93.2, -77.0)
- moved D3 166.3 mm to (113.2, -77.0)
- moved D17 155.5 mm to (73.0, -36.8), turned to 180 degrees
- moved D4 121.0 mm to (113.2, -56.9)
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