File: corne-hotswap/corne-hotswap.kicad_sch (KiCad schematic)
At the start: 61 parts, among them J1 Battery, J2 nice!view, SW1 SW_Push, SW10 SW_Push, SW11 SW_Push, SW12 SW_Push, SW13 SW_Push, SW14 SW_Push, SW15 SW_Push, SW16 SW_Push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

Commit message: Update corne-hotswap.kicad_sch
Parts:
- removed JP1, JP2, JP3, JP4, JP5, JP6: SolderJumper_3_Open, symbol Jumper:SolderJumper_3_Open
- removed U1: nice!nano, symbol Corne:NiceNano
- added J3: OLED display, symbol Connector_Generic:Conn_01x04
- added U1: ProMicro, PCM_marbastlib-xp-promicroish:ProMicro_USBup, symbol PCM_marbastlib-promicroish:Arduino_ProMicro
Connections:
- net CS: now also U1.24 (B6)
- net GND: now also U1.14 (GND), U1.3 (GND), U1.4 (GND)
- net SCK: no longer JP8.2 (B)
- net VCC: now also J3.3 (Pin_3), U1.16 (VCC)
- net col0: now also U1.17 (F4)
- net col1: now also U1.18 (F5)
- net col2: now also U1.19 (F6)
- net col3: now also U1.20 (F7)
- net col4: now also U1.21 (B1)
- net col5: now also U1.22 (B3)
- net raw: now also U1.13 (B0)
- net reset: now also U1.15 (RST)
- net row0: now also U1.7 (D4)
- net row1: now also U1.8 (C6)
- net row2: now also U1.9 (D7)
- net row3: now also U1.10 (E6)
- net jump0: now reaches J2.1 (Pin_1), JP11.1 (A), JP7.1 (A)
- net jump0: now also J3.1 (Pin_1)
- net jump2: now reaches J2.4 (Pin_4), JP13.1 (A), JP9.1 (A)
- net jump2: now also J3.4 (Pin_4)
- net jump1: now reaches J2.2 (Pin_2), JP12.1 (A), JP8.1 (A)
- net jump1: now also J3.2 (Pin_2)
- net jump3: now reaches J2.5 (Pin_5), JP10.1 (A), JP14.1 (A)
- net MOSI renamed SCL
- net SCL: now also JP8.2 (B), U1.6 (D0); no longer JP7.2 (B)
- new net SDA: JP7.2 (B), U1.5 (D1)
- no-connect marks 7 -> 3
Other:
- moved on the sheet: JP10, JP11, JP12, JP13, JP14, JP7, JP8, JP9

Commit message: footprint assign
Parts:
- D1, D10, D11, D12, D13, D14, D15, D16, D17, D18, D19, D2, D20, D21, D3, D4, D5, D6, D7, D8, D9: footprint (none) -> Project:Diode-Reversible
- J1: value Battery -> Battery Connector; footprint (none) -> Connector_JST:JST_PH_S2B-PH-K_1x02_P2.00mm_Horizontal
- J2: footprint (none) -> Project:Nice_View
- J3: footprint (none) -> Project:OLED_Display
- JP10, JP11, JP12, JP13, JP14, JP7, JP8, JP9: footprint (none) -> Jumper:SolderJumper-2_P1.3mm_Open_RoundedPad1.0x1.5mm
- PSW1: footprint (none) -> Button_Switch_SMD:SW_SPDT_PCM12
- RSW1, SW1, SW10, SW11, SW12, SW13, SW14, SW15, SW16, SW17, SW18, SW19, SW2, SW20, SW21, SW3, SW4, SW5, SW6, SW7, SW8, SW9: footprint (none) -> Project:Switch-MX_ChocV2-Reversible-Hotswap
- U1: footprint PCM_marbastlib-xp-promicroish:ProMicro_USBup -> Project:Pro_Micro-Reversible
Changed lines of the file:
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@@
 			)
 		)
-		(property "Footprint" ""
+		(property "Footprint" "Project:Switch-MX_ChocV2-Reversible-Hotswap"
 			(at 191.77 111.76 0)
 			(effects
@@
 			)
 		)
-		(property "Footprint" ""
+		(property "Footprint" "Project:Diode-Reversible"
 			(at 232.41 102.87 0)
 			(effects
@@
 			)
 		)
-		(property "Footprint" ""
+		(property "Footprint" "Project:Switch-MX_ChocV2-Reversible-Hotswap"
 			(at 245.11 129.54 0)
 			(effects
@@
 			)
 		)
-		(property "Value" "Battery"
+		(property "Value" "Battery Connector"
 			(at 73.66 106.6799 0)
 			(effects
@@
 			)
 		)
-		(property "Footprint" ""
+		(property "Footprint" "Connector_JST:JST_PH_S2B-PH-K_1x02_P2.00mm_Horizontal"
 			(at 71.12 104.14 0)
 			(effects
@@
 			)
 		)
-		(property "Footprint" ""
+		(property "Footprint" "Project:Switch-MX_ChocV2-Reversible-Hotswap"
 			(at 262.89 129.54 0)
 			(effects
@@
 			)
 		)
-		(property "Footprint" ""
+		(property "Footprint" "Project:Switch-MX_ChocV2-Reversible-Hotswap"
 			(at 262.89 111.76 0)
 			(effects
@@
 			)
 		)
-		(property "Footprint" ""
+		(property "Footprint" "Project:Diode-Reversible"
 			(at 214.63 120.65 0)
 			(effects
@@
 			)
 		)
-		(property "Footprint" ""
+		(property "Footprint" "Project:Diode-Reversible"
 			(at 250.19 156.21 0)
 			(effects
@@
 			)
 		)
-		(property "Footprint" ""
+		(property "Footprint" "Project:Diode-Reversible"
 			(at 214.63 138.43 0)
 			(effects
@@
 			)
 		)
-		(property "Footprint" ""
+		(property "Footprint" "Project:Diode-Reversible"
 			(at 196.85 120.65 0)
 			(effects
@@
 			)
 		)
-		(property "Footprint" ""
+		(property "Footprint" "Project:Switch-MX_ChocV2-Reversible-Hotswap"
 			(at 227.33 129.54 0)
 			(effects
@@
 			)
 		)
-		(property "Footprint" ""
+		(property "Footprint" "Project:Diode-Reversible"
 			(at 179.07 102.87 0)
 			(effects
@@
 			)
 		)
-		(property "Footprint" ""
+		(property "Footprint" "Project:OLED_Display"
 			(at 128.27 130.81 0)
 			(effects
@@
 			)
 		)
-		(property "Footprint" ""
+		(property "Footprint" "Project:Switch-MX_ChocV2-Reversible-Hotswap"
 			(at 262.89 147.32 0)
 			(effects
@@
 			)
 		)
-		(property "Footprint" ""
+		(property "Footprint" "Project:Diode-Reversible"
 			(at 179.07 138.43 0)
 			(effects
@@
 			)
 		)
-		(property "Footprint" ""
+		(property "Footprint" "Project:Diode-Reversible"
 			(at 179.07 120.65 0)
 			(effects
@@
 			)
 		)
-		(property "Footprint" ""
+		(property "Footprint" "Project:Diode-Reversible"
 			(at 196.85 102.87 0)
 			(effects
@@
 			)
 		)
-		(property "Footprint" ""
+		(property "Footprint" "Project:Switch-MX_ChocV2-Reversible-Hotswap"
 			(at 191.77 93.98 0)
 			(effects
@@
 			)
 		)
-		(property "Footprint" ""
+		(property "Footprint" "Project:Switch-MX_ChocV2-Reversible-Hotswap"
 			(at 191.77 129.54 0)
 			(effects
@@
 			)
 		)
-		(property "Footprint" ""
+		(property "Footprint" "Project:Switch-MX_ChocV2-Reversible-Hotswap"
 			(at 173.99 93.98 0)
 			(effects
@@
 			)
 		)
-		(property "Footprint" ""
+		(property "Footprint" "Project:Diode-Reversible"
 			(at 267.97 102.87 0)
 			(effects
@@
 			)
 		)
-		(property "Footprint" ""
+		(property "Footprint" "Project:Switch-MX_ChocV2-Reversible-Hotswap"
 			(at 173.99 129.54 0)
 			(effects
@@
 			)
 		)
-		(property "Footprint" ""
+		(property "Footprint" "Project:Switch-MX_ChocV2-Reversible-Hotswap"
 			(at 262.89 93.98 0)
 			(effects
@@
 			)
 		)
-		(property "Footprint" ""
+		(property "Footprint" "Project:Diode-Reversible"
 			(at 267.97 138.43 0)
 			(effects
@@
 			)
 		)
-		(property "Footprint" ""
+		(property "Footprint" "Jumper:SolderJumper-2_P1.3mm_Open_RoundedPad1.0x1.5mm"
 			(at 111.76 167.64 0)
 			(effects
@@
 			)
 		)
-		(property "Footprint" ""
+		(property "Footprint" "Project:Switch-MX_ChocV2-Reversible-Hotswap"
 			(at 227.33 111.76 0)
 			(effects
@@
 			)
 		)
-		(property "Footprint" ""
+		(property "Footprint" "Project:Switch-MX_ChocV2-Reversible-Hotswap"
 			(at 245.11 93.98 0)
 			(effects
@@
 			)
 		)
-		(property "Footprint" ""
+		(property "Footprint" "Jumper:SolderJumper-2_P1.3mm_Open_RoundedPad1.0x1.5mm"
 			(at 132.08 177.8 0)
 			(effects
@@
 			)
 		)
-		(property "Footprint" ""
+		(property "Footprint" "Jumper:SolderJumper-2_P1.3mm_Open_RoundedPad1.0x1.5mm"
 			(at 111.76 177.8 0)
 			(effects
@@
 			)
 		)
-		(property "Footprint" ""
+		(property "Footprint" "Project:Nice_View"
 			(at 113.03 130.81 0)
 			(effects
@@
 			)
 		)
-		(property "Footprint" ""
+		(property "Footprint" "Jumper:SolderJumper-2_P1.3mm_Open_RoundedPad1.0x1.5mm"
 			(at 132.08 172.72 0)
 			(effects
@@
 			)
 		)
-		(property "Footprint" ""
+		(property "Footprint" "Project:Switch-MX_ChocV2-Reversible-Hotswap"
 			(at 209.55 111.76 0)
 			(effects
@@
 			)
 		)
-		(property "Footprint" ""
+		(property "Footprint" "Button_Switch_SMD:SW_SPDT_PCM12"
 			(at 53.34 104.14 0)
 			(effects
@@
 			)
 		)
-		(property "Footprint" ""
+		(property "Footprint" "Jumper:SolderJumper-2_P1.3mm_Open_RoundedPad1.0x1.5mm"
 			(at 132.08 167.64 0)
 			(effects
@@
 			)
 		)
-		(property "Footprint" ""
+		(property "Footprint" "Project:Diode-Reversible"
 			(at 214.63 102.87 0)
 			(effects
@@
 			)
 		)
-		(property "Footprint" ""
+		(property "Footprint" "Project:Diode-Reversible"
 			(at 267.97 156.21 0)
 			(effects
@@
 			)
 		)
-		(property "Footprint" ""
+		(property "Footprint" "Project:Switch-MX_ChocV2-Reversible-Hotswap"
 			(at 173.99 111.76 0)
 			(effects
@@
 			)
 		)
-		(property "Footprint" ""
+		(property "Footprint" "Project:Switch-MX_ChocV2-Reversible-Hotswap"
 			(at 227.33 147.32 0)
 			(effects
@@
 			)
 		)
-		(property "Footprint" ""
+		(property "Footprint" "Jumper:SolderJumper-2_P1.3mm_Open_RoundedPad1.0x1.5mm"
 			(at 111.76 182.88 0)
 			(effects
@@
 			)
 		)
-		(property "Footprint" ""
+		(property "Footprint" "Project:Switch-MX_ChocV2-Reversible-Hotswap"
 			(at 245.11 111.76 0)
 			(effects
@@
 			)
 		)
-		(property "Footprint" ""
+		(property "Footprint" "Project:Diode-Reversible"
 			(at 232.41 120.65 0)
 			(effects
@@
 			)
 		)
-		(property "Footprint" ""
+		(property "Footprint" "Project:Diode-Reversible"
 			(at 250.19 138.43 0)
 			(effects
@@
 			)
 		)
-		(property "Footprint" ""
+		(property "Footprint" "Project:Switch-MX_ChocV2-Reversible-Hotswap"
 			(at 209.55 129.54 0)
 			(effects
@@
 			)
 		)
-		(property "Footprint" ""
+		(property "Footprint" "Project:Diode-Reversible"
 			(at 232.41 156.21 0)
 			(effects
@@
 			)
 		)
-		(property "Footprint" ""
+		(property "Footprint" "Jumper:SolderJumper-2_P1.3mm_Open_RoundedPad1.0x1.5mm"
 			(at 132.08 182.88 0)
 			(effects
@@
 			)
 		)
-		(property "Footprint" "PCM_marbastlib-xp-promicroish:ProMicro_USBup"
+		(property "Footprint" "Project:Pro_Micro-Reversible"
 			(at 58.42 93.98 0)
 			(effects
@@
 			)
 		)
-		(property "Footprint" ""
+		(property "Footprint" "Project:Switch-MX_ChocV2-Reversible-Hotswap"
 			(at 209.55 93.98 0)
 			(effects
@@
 			)
 		)
-		(property "Footprint" ""
+		(property "Footprint" "Project:Switch-MX_ChocV2-Reversible-Hotswap"
 			(at 245.11 147.32 0)
 			(effects
@@
 			)
 		)
-		(property "Footprint" ""
+		(property "Footprint" "Project:Diode-Reversible"
 			(at 267.97 120.65 0)
 			(effects
@@
 			)
 		)
-		(property "Footprint" ""
+		(property "Footprint" "Project:Switch-MX_ChocV2-Reversible-Hotswap"
 			(at 227.33 93.98 0)
 			(effects
@@
 			)
 		)
-		(property "Footprint" ""
+		(property "Footprint" "Project:Diode-Reversible"
 			(at 196.85 138.43 0)
 			(effects
@@
 			)
 		)
-		(property "Footprint" ""
+		(property "Footprint" "Jumper:SolderJumper-2_P1.3mm_Open_RoundedPad1.0x1.5mm"
 			(at 111.76 172.72 0)
 			(effects
@@
 			)
 		)
-		(property "Footprint" ""
+		(property "Footprint" "Project:Diode-Reversible"
 			(at 250.19 102.87 0)
 			(effects
@@
 			)
 		)
-		(property "Footprint" ""
+		(property "Footprint" "Project:Diode-Reversible"
 			(at 250.19 120.65 0)
 			(effects
@@
 			)
 		)
-		(property "Footprint" ""
+		(property "Footprint" "Project:Diode-Reversible"
 			(at 232.41 138.43 0)
 			(effects
@@
 			)
 		)
-		(property "Footprint" ""
+		(property "Footprint" "Project:Switch-MX_ChocV2-Reversible-Hotswap"
 			(at 53.34 118.11 0)
 			(effects

Commit message: remove wrong footprint from reset switch
Parts:
- RSW1: footprint Project:Switch-MX_ChocV2-Reversible-Hotswap -> (none)
Changed lines of the file:
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@@
 			)
 		)
-		(property "Footprint" "Project:Switch-MX_ChocV2-Reversible-Hotswap"
+		(property "Footprint" ""
 			(at 53.34 118.11 0)
 			(effects

Commit message: pcb edit
Parts:
- PSW1: footprint Button_Switch_SMD:SW_SPDT_PCM12 -> Project:SW_SPDT_PCM12
- RSW1: footprint (none) -> Project:SW_PUSH_1P1T_6x3.5mm_H4.3_APEM_MJTP1243
Connections:
- net CS: now also U1.12 (B5); no longer U1.24 (B6)
- net raw renamed RAW
- net reset renamed RST
Changed lines of the file:
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@@
 		)
 	)
-	(global_label "reset"
+	(global_label "RST"
 		(shape input)
 		(at 58.42 123.19 0)
@@
 		)
 		(property "Intersheetrefs" "${INTERSHEET_REFS}"
-			(at 66.1224 123.19 0)
+			(at 64.8523 123.19 0)
 			(effects
 				(font
@@
 		)
 	)
-	(global_label "raw"
+	(global_label "RAW"
 		(shape input)
 		(at 71.12 49.53 0)
@@
 		)
 		(property "Intersheetrefs" "${INTERSHEET_REFS}"
-			(at 77.3709 49.53 0)
+			(at 77.9152 49.53 0)
 			(effects
 				(font
@@
 		)
 	)
-	(global_label "raw"
+	(global_label "RAW"
 		(shape input)
 		(at 48.26 106.68 180)
@@
 		)
 		(property "Intersheetrefs" "${INTERSHEET_REFS}"
-			(at 42.0091 106.68 0)
+			(at 41.4648 106.68 0)
 			(effects
 				(font
@@
 		)
 	)
-	(global_label "jump3"
+	(global_label "CS"
 		(shape input)
-		(at 118.11 135.89 270)
+		(at 45.72 77.47 180)
 		(fields_autoplaced yes)
 		(effects
@@
 		)
 		(property "Intersheetrefs" "${INTERSHEET_REFS}"
-			(at 118.11 144.6808 90)
+			(at 40.2553 77.47 0)
 			(effects
 				(font
@@
 		)
 	)
-	(global_label "jump2"
+	(global_label "jump3"
 		(shape input)
-		(at 123.19 161.29 90)
+		(at 118.11 135.89 270)
 		(fields_autoplaced yes)
 		(effects
@@
 				(size 1.27 1.27)
 			)
-			(justify left)
+			(justify right)
 		)
 		(property "Intersheetrefs" "${INTERSHEET_REFS}"
-			(at 123.19 152.4992 90)
+			(at 118.11 144.6808 90)
 			(effects
 				(font
 					(size 1.27 1.27)
 				)
-				(justify left)
+				(justify right)
 				(hide yes)
 			)
 		)
 	)
-	(global_label "row0"
+	(global_label "jump2"
 		(shape input)
-		(at 45.72 64.77 180)
+		(at 123.19 161.29 90)
 		(fields_autoplaced yes)
 		(effects
@@
 				(size 1.27 1.27)
 			)
-			(justify right)
+			(justify left)
 		)
 		(property "Intersheetrefs" "${INTERSHEET_REFS}"
-			(at 38.2596 64.77 0)
+			(at 123.19 152.4992 90)
 			(effects
 				(font
 					(size 1.27 1.27)
 				)
-				(justify right)
+				(justify left)
 				(hide yes)
 			)
 		)
 	)
-	(global_label "CS"
+	(global_label "row0"
 		(shape input)
-		(at 71.12 77.47 0)
+		(at 45.72 64.77 180)
 		(fields_autoplaced yes)
 		(effects
@@
 				(size 1.27 1.27)
 			)
-			(justify left)
+			(justify right)
 		)
 		(property "Intersheetrefs" "${INTERSHEET_REFS}"
-			(at 76.5847 77.47 0)
+			(at 38.2596 64.77 0)
 			(effects
 				(font
 					(size 1.27 1.27)
 				)
-				(justify left)
+				(justify right)
 				(hide yes)
 			)
 		)
 	)
-	(global_label "reset"
+	(global_label "RST"
 		(shape input)
 		(at 71.12 54.61 0)
@@
 		)
 		(property "Intersheetrefs" "${INTERSHEET_REFS}"
-			(at 78.8224 54.61 0)
+			(at 77.5523 54.61 0)
 			(effects
 				(font
@@
 			)
 		)
-		(property "Footprint" "Button_Switch_SMD:SW_SPDT_PCM12"
+		(property "Footprint" "Project:SW_SPDT_PCM12"
 			(at 53.34 104.14 0)
 			(effects
@@
 			)
 		)
-		(property "Footprint" ""
+		(property "Footprint" "Project:SW_PUSH_1P1T_6x3.5mm_H4.3_APEM_MJTP1243"
 			(at 53.34 118.11 0)
 			(effects

Commit message: update
Parts:
- removed J3: OLED display, Project:OLED_Display, symbol Connector_Generic:Conn_01x04
- removed JP10, JP11, JP12, JP13, JP14, JP7, JP8, JP9: SolderJumper_2_Open, Jumper:SolderJumper-2_P1.3mm_Open_RoundedPad1.0x1.5mm, symbol Jumper:SolderJumper_2_Open
- D1, D10, D11, D12, D13, D14, D15, D16, D17, D18, D19, D2, D20, D21, D3, D4, D5, D6, D7, D8, D9: footprint Project:Diode-Reversible -> Project:D_SOD-123F-Reversible
Connections:
- net jump0 is gone; now on net SDA: J2.1 (Pin_1)
- net jump1 is gone; now on net SCL: J2.2 (Pin_2)
- net jump2 is gone; now on net GND: J2.4 (Pin_4)
- net jump3 is gone; now on net CS: J2.5 (Pin_5)
Other:
- moved on the sheet: J2

Commit message: edit
Parts:
- D1, D10, D11, D12, D13, D14, D15, D16, D17, D18, D19, D2, D20, D21, D3, D4, D5, D6, D7, D8, D9: footprint Project:D_SOD-123F-Reversible -> Project:D_SOD-123F-Reversible-Hotswap
Changed lines of the file:
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@@
 			)
 		)
-		(property "Footprint" "Project:D_SOD-123F-Reversible"
+		(property "Footprint" "Project:D_SOD-123F-Reversible-Hotswap"
 			(at 232.41 102.87 0)
 			(effects
@@
 			)
 		)
-		(property "Footprint" "Project:D_SOD-123F-Reversible"
+		(property "Footprint" "Project:D_SOD-123F-Reversible-Hotswap"
 			(at 214.63 120.65 0)
 			(effects
@@
 			)
 		)
-		(property "Footprint" "Project:D_SOD-123F-Reversible"
+		(property "Footprint" "Project:D_SOD-123F-Reversible-Hotswap"
 			(at 250.19 156.21 0)
 			(effects
@@
 			)
 		)
-		(property "Footprint" "Project:D_SOD-123F-Reversible"
+		(property "Footprint" "Project:D_SOD-123F-Reversible-Hotswap"
 			(at 214.63 138.43 0)
 			(effects
@@
 			)
 		)
-		(property "Footprint" "Project:D_SOD-123F-Reversible"
+		(property "Footprint" "Project:D_SOD-123F-Reversible-Hotswap"
 			(at 196.85 120.65 0)
 			(effects
@@
 			)
 		)
-		(property "Footprint" "Project:D_SOD-123F-Reversible"
+		(property "Footprint" "Project:D_SOD-123F-Reversible-Hotswap"
 			(at 179.07 102.87 0)
 			(effects
@@
 			)
 		)
-		(property "Footprint" "Project:D_SOD-123F-Reversible"
+		(property "Footprint" "Project:D_SOD-123F-Reversible-Hotswap"
 			(at 179.07 138.43 0)
 			(effects
@@
 			)
 		)
-		(property "Footprint" "Project:D_SOD-123F-Reversible"
+		(property "Footprint" "Project:D_SOD-123F-Reversible-Hotswap"
 			(at 179.07 120.65 0)
 			(effects
@@
 			)
 		)
-		(property "Footprint" "Project:D_SOD-123F-Reversible"
+		(property "Footprint" "Project:D_SOD-123F-Reversible-Hotswap"
 			(at 196.85 102.87 0)
 			(effects
@@
 			)
 		)
-		(property "Footprint" "Project:D_SOD-123F-Reversible"
+		(property "Footprint" "Project:D_SOD-123F-Reversible-Hotswap"
 			(at 267.97 102.87 0)
 			(effects
@@
 			)
 		)
-		(property "Footprint" "Project:D_SOD-123F-Reversible"
+		(property "Footprint" "Project:D_SOD-123F-Reversible-Hotswap"
 			(at 267.97 138.43 0)
 			(effects
@@
 			)
 		)
-		(property "Footprint" "Project:D_SOD-123F-Reversible"
+		(property "Footprint" "Project:D_SOD-123F-Reversible-Hotswap"
 			(at 214.63 102.87 0)
 			(effects
@@
 			)
 		)
-		(property "Footprint" "Project:D_SOD-123F-Reversible"
+		(property "Footprint" "Project:D_SOD-123F-Reversible-Hotswap"
 			(at 267.97 156.21 0)
 			(effects
@@
 			)
 		)
-		(property "Footprint" "Project:D_SOD-123F-Reversible"
+		(property "Footprint" "Project:D_SOD-123F-Reversible-Hotswap"
 			(at 232.41 120.65 0)
 			(effects
@@
 			)
 		)
-		(property "Footprint" "Project:D_SOD-123F-Reversible"
+		(property "Footprint" "Project:D_SOD-123F-Reversible-Hotswap"
 			(at 250.19 138.43 0)
 			(effects
@@
 			)
 		)
-		(property "Footprint" "Project:D_SOD-123F-Reversible"
+		(property "Footprint" "Project:D_SOD-123F-Reversible-Hotswap"
 			(at 232.41 156.21 0)
 			(effects
@@
 			)
 		)
-		(property "Footprint" "Project:D_SOD-123F-Reversible"
+		(property "Footprint" "Project:D_SOD-123F-Reversible-Hotswap"
 			(at 267.97 120.65 0)
 			(effects
@@
 			)
 		)
-		(property "Footprint" "Project:D_SOD-123F-Reversible"
+		(property "Footprint" "Project:D_SOD-123F-Reversible-Hotswap"
 			(at 196.85 138.43 0)
 			(effects
@@
 			)
 		)
-		(property "Footprint" "Project:D_SOD-123F-Reversible"
+		(property "Footprint" "Project:D_SOD-123F-Reversible-Hotswap"
 			(at 250.19 102.87 0)
 			(effects
@@
 			)
 		)
-		(property "Footprint" "Project:D_SOD-123F-Reversible"
+		(property "Footprint" "Project:D_SOD-123F-Reversible-Hotswap"
 			(at 250.19 120.65 0)
 			(effects
@@
 			)
 		)
-		(property "Footprint" "Project:D_SOD-123F-Reversible"
+		(property "Footprint" "Project:D_SOD-123F-Reversible-Hotswap"
 			(at 232.41 138.43 0)
 			(effects
