File: corne-hotswap-wip/corne-hotswap.kicad_pcb (KiCad board)
At the start: 2 copper layers, 133.8 x 91.7 mm, 49 parts, among them J1 Battery Connector, J2 nice!view, J3 USB_C_Receptacle_PowerOnly_6P, J4 Battery Wire, SW1 SW_Push, SW10 SW_Push, SW11 SW_Push, SW12 SW_Push, SW13 SW_Push, SW14 SW_Push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

Commit message: column wiring
Routing:
- net col4: track 0.00 -> 43.0 mm
- net col3: track 0.00 -> 36.0 mm
- net col5: track 0.00 -> 31.6 mm
- net col0: track 12.0 -> 31.0 mm
- net col2: track 0.00 -> 19.0 mm
- net col1: track 12.0 -> 31.0 mm
- net Net-(D21-A): track 0.00 -> 18.0 mm
- net Net-(D17-A): track 0.00 -> 4.30 mm
- net Net-(D9-A): track 0.00 -> 3.86 mm
- net Net-(D8-A): track 0.00 -> 3.86 mm
- net Net-(D7-A): track 0.00 -> 3.86 mm
- net Net-(D6-A): track 0.00 -> 3.86 mm
- net Net-(D5-A): track 0.00 -> 3.86 mm
- net Net-(D4-A): track 0.00 -> 3.86 mm
- net Net-(D3-A): track 0.00 -> 3.86 mm
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
Commit message: wiring
Routing:
- net row0: track 0.00 -> 119.3 mm
- net col0: track 31.0 -> 141.3 mm
- net col2: track 19.0 -> 128.8 mm
- net row2: track 0.00 -> 109.3 mm
- net row1: track 0.00 -> 102.3 mm
- net col1: track 31.0 -> 131.4 mm
- net col3: track 36.0 -> 121.8 mm
- net col4: track 43.0 -> 103.8 mm
- net row3: track 0.00 -> 59.9 mm
- net col5: track 31.6 -> 82.2 mm, vias 0 -> 2

Commit message: Update corne-hotswap.kicad_pcb
Routing:
- net col0: track 141.3 -> 146.2 mm
- net col5: track 82.2 -> 85.8 mm, vias 2 -> 0
- net col2: track 128.8 -> 131.1 mm
- net col1: track 131.4 -> 133.2 mm
- net row1: track 102.3 -> 102.7 mm, vias 0 -> 1
- net row2: track 109.3 -> 109.1 mm, vias 0 -> 1
- net GND: vias 3 -> 21

Commit message: Update corne-hotswap.kicad_pcb
Routing:
- net row1: track 102.7 -> 106.2 mm
- net row0: track 119.3 -> 120.2 mm
- net row3: track 59.9 -> 60.7 mm
- net col3: track 121.8 -> 121.3 mm
- net GND: vias 21 -> 24
