File: corne-module/corne-module.kicad_pcb (KiCad board)
At the start: 2 copper layers, 16.6 x 10.7 mm, 7 parts, among them J1 Battery Connector, J2 nice!view, J3 USB_C_Receptacle_PowerOnly_6P, J4 Battery Wire, U1 ProMicro

Commit message: edit jumpers and texts
Routing:
- net GND: track 100.7 -> 101.4 mm
